Commit message: update gp4 and rendering scripts

File: assets/gp4_lego/gp4.urdf (robot description, URDF)
Before this commit: robot Yaskawa_gp4, 12 links, 11 joints
Links:
- link fts: geometry collision cylinder length=0.0505 radius=0.048; visual cylinder length=0.0505 radius=0.0472
Joints:
- joint joint_3: limit lower=-1.1344640137963142 upper=3.490658503988659 effort=200 velocity=2 -> lower=-0.99 upper=3.30 effort=200 velocity=2

File: assets/gp4_lego/gp4_spherized.urdf (robot description, URDF)
Before this commit: robot Yaskawa_gp4, 12 links, 11 joints
Links:
- link base_link: geometry collision sphere radius=0.013025; collision sphere radius=0.014502
- link fts: geometry collision sphere radius=0.007188; collision sphere radius=0.007966
- link link_1: geometry collision sphere radius=0.013918; collision sphere radius=0.014057
- link link_3: geometry collision sphere radius=0.001891; collision sphere radius=0.017254
- link link_5: geometry collision sphere radius=0.008942; collision sphere radius=0.009298
- link link_tool: geometry collision sphere radius=0.000103; collision sphere radius=0.000178
Joints:
- joint joint_3: limit lower=-1.1344640137963142 upper=3.490658503988659 effort=200 velocity=2 -> lower=-0.99 upper=3.30 effort=200 velocity=2

File: assets/gp4_lego/gp4_spherized_visual_from_collision.urdf (robot description, URDF)
Before this commit: robot Yaskawa_gp4, 12 links, 11 joints
Links:
- link base_link: geometry collision sphere radius=0.013025; collision sphere radius=0.014502
- link fts: geometry collision sphere radius=0.007188; collision sphere radius=0.007966
- link link_1: geometry collision sphere radius=0.013918; collision sphere radius=0.014057
- link link_3: geometry collision sphere radius=0.001891; collision sphere radius=0.017254
- link link_5: geometry collision sphere radius=0.008942; collision sphere radius=0.009298
- link link_tool: geometry collision sphere radius=0.000103; collision sphere radius=0.000178
Joints:
- joint joint_3: limit lower=-1.1344640137963142 upper=3.490658503988659 effort=200 velocity=2 -> lower=-0.99 upper=3.30 effort=200 velocity=2
